File: EVE-3A keyboard ortho/EVE-3A keyboard ortho.kicad_pcb (KiCad board)
At the start: 2 copper layers, 313.5 x 133 mm, 128 parts, among them J1 Conn_01x04_Male, J2 Conn_01x06_Male, SW1 1, SW10 W, SW11 S, SW12 X, SW13 4, SW14 E, SW15 D, SW16 C, SW17 5, SW18 R, SW19 F, SW2 Esc, SW20 V, SW21 6, SW22 T, SW23 G, SW24 B, SW25 Space, SW26 7, SW27 Y, SW28 H, SW29 N, SW3 Ctrl, SW30 Space, SW31 8, SW32 U, SW33 J, SW34 M, SW35 Space, SW36 9, SW37 I, SW38 K, SW39 ,, SW4 ShiftL, SW40 0, SW41 O, SW42 L, SW43 ., SW44 :, SW45 P, SW46 ;, SW47 /, SW48 - =, SW49 LineFeed, SW5 2, SW50 @, SW51 ShiftR, SW52 [, SW53 Enter, SW54 \, SW55 ], SW56 _ Rub, SW57 Repeat, SW58 ^ ~ Home, SW59 Here Is, SW6 Q, SW60 Break, SW61 Clear, SW62 Special, SW7 A, SW8 Z, SW9 3, U1 74LS138, U2 74LS138

Commit message: interim checkin
Parts:
- removed J2: Conn_01x06_Male, Connector_PinHeader_2.54mm:PinHeader_1x06_P2.54mm_Horizontal
- J1: value Conn_01x04_Male -> Conn_02x04_Odd_Even; footprint Connector_PinHeader_2.54mm:PinHeader_1x04_P2.54mm_Horizontal -> Connector_IDC:IDC-Header_2x04_P2.54mm_Vertical
- U1, U2: value 74LS138 -> 74LS595
- moved C2 117.8 mm to (231.0, 43.2), turned to -90 degrees
- moved U2 99.5 mm to (220.9, 48.3), turned to 90 degrees
- moved U1 95.9 mm to (182.8, 48.3), turned to 90 degrees
- moved J1 89.2 mm to (76.1, 43.2)
- moved C1 88.9 mm to (154.8, 43.2), turned to -90 degrees
- moved D1 77.6 mm to (54.5, 66.7)
- moved D10 77.6 mm to (92.5, 85.7)
- moved D11 77.6 mm to (92.5, 104.7)
- moved D12 77.6 mm to (92.5, 123.7)
- moved D13 77.6 mm to (111.5, 66.7)
- moved D14 77.6 mm to (111.5, 85.7)
- moved D15 77.6 mm to (111.5, 104.7)
- moved D16 77.6 mm to (111.5, 123.7)
- moved D17 77.6 mm to (130.5, 66.7)
- moved D18 77.6 mm to (130.5, 85.7)
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Connections:
- D33 pad 1: Net-(U2-Pad10) -> Net-(D33-Pad1)
- D42 pad 1: Net-(U2-Pad12) -> Net-(D42-Pad1)
- D43 pad 1: Net-(U2-Pad12) -> Net-(D42-Pad1)
- D44 pad 1: Net-(U2-Pad12) -> Net-(D42-Pad1)
- D45 pad 1: Net-(U2-Pad12) -> Net-(D42-Pad1)
- D46 pad 1: Net-(U2-Pad11) -> Net-(D46-Pad1)
- D47 pad 1: Net-(U2-Pad11) -> Net-(D46-Pad1)
- D48 pad 1: Net-(U2-Pad11) -> Net-(D46-Pad1)
- D49 pad 1: Net-(U2-Pad11) -> Net-(D46-Pad1)
- D50 pad 1: Net-(U2-Pad10) -> Net-(D33-Pad1)
- D51 pad 1: Net-(U2-Pad10) -> Net-(D33-Pad1)
- D52 pad 1: Net-(U2-Pad10) -> Net-(D33-Pad1)
- D53 pad 1: Net-(U2-Pad9) -> Net-(D53-Pad1)
- D54 pad 1: Net-(U2-Pad9) -> Net-(D53-Pad1)
- D55 pad 1: Net-(U2-Pad9) -> Net-(D53-Pad1)
- D56 pad 1: Net-(U2-Pad7) -> Net-(D56-Pad1)
- D57 pad 1: Net-(U2-Pad7) -> Net-(D56-Pad1)
- D58 pad 1: Net-(U2-Pad7) -> Net-(D56-Pad1)
- D59 pad 1: Net-(U2-Pad7) -> Net-(D56-Pad1)
- D60 pad 1: Net-(U2-Pad9) -> Net-(D53-Pad1)
- J1 pad 2: R1 -> Net-(U1-Pad10)
- J1 pad 3: R2 -> R1
- J1 pad 4: R3 -> Net-(U2-Pad14)
- U1 pad 1: C0 -> Net-(D25-Pad1)
- U1 pad 10: Net-(D21-Pad1) -> Net-(U1-Pad10)
- U1 pad 11: Net-(D17-Pad1) -> Net-(U1-Pad10)
- U1 pad 12: Net-(D13-Pad1) -> GND
- U1 pad 13: Net-(D10-Pad1) -> GND
- U1 pad 14: Net-(D5-Pad1) -> Net-(U1-Pad14)
- U1 pad 15: Net-(D1-Pad1) -> Net-(D29-Pad1)
- U1 pad 2: C1 -> Net-(D21-Pad1)
- U1 pad 3: C2 -> Net-(D17-Pad1)
- U1 pad 4: GND -> Net-(D13-Pad1)
- U1 pad 5: GND -> Net-(D10-Pad1)
- U1 pad 6: C3 -> Net-(D5-Pad1)
- U1 pad 7: Net-(D29-Pad1) -> Net-(D1-Pad1)
- U1 pad 9: Net-(D25-Pad1) -> unconnected-(U1-Pad9)
- U2 pad 1: C0 -> Net-(D56-Pad1)
- U2 pad 10: Net-(U2-Pad10) -> Net-(U1-Pad10)
- U2 pad 11: Net-(U2-Pad11) -> Net-(U1-Pad10)
- U2 pad 12: Net-(U2-Pad12) -> GND
- U2 pad 13: Net-(D38-Pad1) -> GND
- U2 pad 14: Net-(D34-Pad1) -> Net-(U2-Pad14)
- U2 pad 2: C1 -> Net-(D53-Pad1)
- U2 pad 3: C2 -> Net-(D33-Pad1)
- U2 pad 4: GND -> Net-(D46-Pad1)
- U2 pad 5: C3 -> Net-(D42-Pad1)
- U2 pad 6: +3V3 -> Net-(D38-Pad1)
- U2 pad 7: Net-(U2-Pad7) -> Net-(D34-Pad1)
- U2 pad 9: Net-(U2-Pad9) -> Net-(U1-Pad14)
Routing:
- net R3: track 0.00 -> 275.6 mm
- net Net-(U2-Pad14): track 0.00 -> 147.3 mm
- net Net-(U1-Pad10): track 0.00 -> 144.8 mm
- net Net-(D33-Pad1): track 0.00 -> 85.9 mm
- net Net-(D56-Pad1): track 0.00 -> 70.3 mm
- net Net-(D5-Pad1): track 0.00 -> 70.3 mm
- net Net-(D46-Pad1): track 0.00 -> 70.3 mm
- net Net-(D42-Pad1): track 0.00 -> 70.3 mm
- net Net-(D38-Pad1): track 0.00 -> 70.3 mm
- net Net-(D34-Pad1): track 0.00 -> 70.3 mm
- net Net-(D29-Pad1): track 0.00 -> 70.3 mm
- net Net-(D25-Pad1): track 0.00 -> 70.3 mm
- net Net-(D21-Pad1): track 0.00 -> 70.3 mm
- net Net-(D17-Pad1): track 0.00 -> 70.3 mm
- net Net-(D13-Pad1): track 0.00 -> 70.3 mm
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- added copper zone on F.Cu, net +3V3
- added copper zone on B.Cu, net GND
Other:
- board outline removed
- board text added: "K"

Commit message: Completed first draft of Ortholinear layout. Removed old layout that is not up to date with new schematics.
Parts:
- added H1: MountingHole_Pad, MountingHole:MountingHole_3.2mm_M3_Pad_Via, F.Cu at (50.7, 152.2)
- added H2: MountingHole_Pad, MountingHole:MountingHole_3.2mm_M3_Pad_Via, F.Cu at (316.7, 38.2)
- added H3: MountingHole_Pad, MountingHole:MountingHole_3.2mm_M3_Pad_Via, F.Cu at (136.2, 152.2)
- added H4: MountingHole_Pad, MountingHole:MountingHole_3.2mm_M3_Pad_Via, F.Cu at (316.7, 152.2)
- added H5: MountingHole_Pad, MountingHole:MountingHole_3.2mm_M3_Pad_Via, F.Cu at (50.7, 38.2)
- added H6: MountingHole_Pad, MountingHole:MountingHole_3.2mm_M3_Pad_Via, F.Cu at (231.2, 152.2)
- added H7: MountingHole_Pad, MountingHole:MountingHole_3.2mm_M3_Pad_Via, F.Cu at (231.2, 38.2)
- added H8: MountingHole_Pad, MountingHole:MountingHole_3.2mm_M3_Pad_Via, F.Cu at (136.2, 38.2)
- added REF**: Stabilizer_Cherry_MX_2.00u, KeysStable:Stabilizer_Cherry_MX_2.00u, F.Cu at (288.2, 95.2)
- added REF**: Stabilizer_Cherry_MX_2.00u, KeysStable:Stabilizer_Cherry_MX_2.00u, F.Cu at (269.2, 133.2)
- added REF**: Stabilizer_Cherry_MX_6.25u, KeysStable:Stabilizer_Cherry_MX_6.25u, F.Cu at (155.2, 152.2)
- moved C1 51.1 mm to (104.0, 48.3)
- moved U1 51.1 mm to (132.0, 53.3)
- moved U2 48.5 mm to (269.1, 53.3)
- moved D33 42.5 mm to (244.5, 142.7)
- moved D52 19.4 mm to (278.7, 123.7)
- moved D54 19.0 mm to (301.5, 123.7)
- moved D55 19.0 mm to (301.5, 142.7)
- moved C2 11.4 mm to (241.2, 48.3)
- moved J1 5.08 mm to (76.1, 48.3)
- moved D49 4.75 mm to (268.2, 123.7)
Connections:
- J1 pad 2: Net-(U1-Pad10) -> Net-(J1-Pad2)
- J1 pad 4: Net-(U2-Pad14) -> Net-(J1-Pad4)
- J1 pad 6: unconnected-(J1-Pad6) -> GND
- J1 pad 8: unconnected-(J1-Pad8) -> +3V3
- U1 pad 10: Net-(U1-Pad10) -> Net-(J1-Pad4)
- U1 pad 11: Net-(U1-Pad10) -> Net-(J1-Pad4)
- U2 pad 10: Net-(U1-Pad10) -> Net-(J1-Pad4)
- U2 pad 11: Net-(U1-Pad10) -> Net-(J1-Pad4)
- U2 pad 14: Net-(U2-Pad14) -> Net-(J1-Pad2)
Routing:
- net R1: track 0.00 -> 415.3 mm, vias 0 -> 2
- net R2: track 0.00 -> 368.6 mm, vias 0 -> 2
- net R0: track 0.00 -> 343.5 mm
- net R3: track 275.6 -> 500.0 mm, vias 0 -> 2
- net Net-(J1-Pad4): track 0.00 -> 193.0 mm
- net Net-(J1-Pad2): track 0.00 -> 193.0 mm
- net Net-(U2-Pad14): track 147.3 -> 0.00 mm
- net Net-(U1-Pad10): track 144.8 -> 0.00 mm
- net Net-(D33-Pad2): track 0.00 -> 138.7 mm
- net Net-(U1-Pad14): track 30.5 -> 129.5 mm
- net Net-(D33-Pad1): track 85.9 -> 179.9 mm
- net Net-(D29-Pad1): track 70.3 -> 146.4 mm
- net Net-(D1-Pad1): track 70.3 -> 136.3 mm
- net Net-(D53-Pad1): track 66.9 -> 128.6 mm
- net Net-(D56-Pad1): track 70.3 -> 130.2 mm
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- added copper zone on F.Cu, net GND
Other:
- board outline added: 289.8 x 135.4 mm
