File: EVE-3A keyboard original layout/EVE-3A keyboard original layout.kicad_sch (KiCad schematic)
At the start: 135 parts, among them J1 Conn_02x04_Odd_Even, SW1 1, SW10 W, SW11 S, SW12 X, SW13 4, SW14 E, SW15 D, SW16 C, SW17 5, SW18 R, SW19 F, SW2 Esc, SW20 V, SW21 6, SW22 T, SW23 G, SW24 B, SW25 Space, SW26 7, SW27 Y, SW28 H, SW29 N, SW3 Ctrl, SW30 Space, SW31 8, SW32 U, SW33 J, SW34 M, SW35 Space, SW36 9, SW37 I, SW38 K, SW39 ,, SW4 ShiftL, SW40 0, SW41 O, SW42 L, SW43 ., SW44 :, SW45 P, SW46 ;, SW47 /, SW48 - =, SW49 LineFeed, SW5 2, SW50 @, SW51 ShiftR, SW52 [, SW53 Enter, SW54 \, SW55 ], SW56 _ Rub, SW57 Repeat, SW58 ^ ~ Home, SW59 Here Is, SW6 Q, SW60 Break, SW61 Clear, SW62 Special, SW7 A, SW8 Z, SW9 3, U1 74LS595, U2 74LS595

Commit message: First draft of Original Layout
Parts:
- added Stab1: Stabelizer Enter, KeysStable:Stabilizer_Cherry_MX_2.00u, symbol Mechanical:MountingHole
- added Stab2: Stabelizer Spacebar, KeysStable:Stabilizer_Cherry_MX_6.00u, symbol Mechanical:MountingHole
- SW25, SW35, SW51: footprint Keys:SW_Hybrid_Cherry_MX_Alps_2.00u -> Keys:SW_Hybrid_Cherry_MX_Alps_1.50u
- SW30: footprint Keys:SW_Hybrid_Cherry_MX_Alps_2.00u -> Keys:SW_Hybrid_Cherry_MX_Alps_6.50u
- SW4: footprint Keys:SW_Hybrid_Cherry_MX_Alps_1.00u -> Keys:SW_Hybrid_Cherry_MX_Alps_1.50u
Changed lines of the file:
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@@
     (pin "2")
+  )
+  (symbol (lib_id "Mechanical:MountingHole") (at 59.69 184.15 0) (unit 1)
+    (in_bom yes) (on_board yes) (fields_autoplaced)
+    (property "Reference" "Stab2" (id 0) (at 62.23 182.8799 0)
+      (effects (font (size 1.27 1.27)) (justify left))
+    )
+    (property "Value" "Stabelizer Spacebar" (id 1) (at 62.23 185.4199 0)
+      (effects (font (size 1.27 1.27)) (justify left))
+    )
+    (property "Footprint" "KeysStable:Stabilizer_Cherry_MX_6.00u" (id 2) (at 59.69 184.15 0)
+      (effects (font (size 1.27 1.27)) hide)
+    )
+    (property "Datasheet" "~" (id 3) (at 59.69 184.15 0)
+      (effects (font (size 1.27 1.27)) hide)
+    )
   )
   (symbol (lib_id "Switch:SW_Push_45deg") (at 217.17 102.87 270) (mirror x) (unit 1)
@@
       (effects (font (size 1.27 1.27)) (justify left))
     )
-    (property "Footprint" "Keys:SW_Hybrid_Cherry_MX_Alps_2.00u" (id 2) (at 118.11 153.67 0)
+    (property "Footprint" "Keys:SW_Hybrid_Cherry_MX_Alps_6.50u" (id 2) (at 118.11 153.67 0)
       (effects (font (size 1.27 1.27)) hide)
     )
@@
     (pin "1")
     (pin "2")
+  )
+  (symbol (lib_id "Mechanical:MountingHole") (at 59.69 176.53 0) (unit 1)
+    (in_bom yes) (on_board yes) (fields_autoplaced)
+    (property "Reference" "Stab1" (id 0) (at 62.23 175.2599 0)
+      (effects (font (size 1.27 1.27)) (justify left))
+    )
+    (property "Value" "Stabelizer Enter" (id 1) (at 62.23 177.7999 0)
+      (effects (font (size 1.27 1.27)) (justify left))
+    )
+    (property "Footprint" "KeysStable:Stabilizer_Cherry_MX_2.00u" (id 2) (at 59.69 176.53 0)
+      (effects (font (size 1.27 1.27)) hide)
+    )
+    (property "Datasheet" "~" (id 3) (at 59.69 176.53 0)
+      (effects (font (size 1.27 1.27)) hide)
+    )
   )
   (symbol (lib_id "Diode:1N4148") (at 208.28 144.78 0) (mirror y) (unit 1)
@@
       (effects (font (size 1.27 1.27)) (justify left))
     )
-    (property "Footprint" "Keys:SW_Hybrid_Cherry_MX_Alps_2.00u" (id 2) (at 101.6 153.67 0)
+    (property "Footprint" "Keys:SW_Hybrid_Cherry_MX_Alps_1.50u" (id 2) (at 101.6 153.67 0)
       (effects (font (size 1.27 1.27)) hide)
     )
@@
       (effects (font (size 1.27 1.27)) (justify left))
     )
-    (property "Footprint" "Keys:SW_Hybrid_Cherry_MX_Alps_1.00u" (id 2) (at 19.05 140.97 0)
+    (property "Footprint" "Keys:SW_Hybrid_Cherry_MX_Alps_1.50u" (id 2) (at 19.05 140.97 0)
       (effects (font (size 1.27 1.27)) hide)
     )
@@
       (effects (font (size 1.27 1.27)) (justify left))
     )
-    (property "Footprint" "Keys:SW_Hybrid_Cherry_MX_Alps_2.00u" (id 2) (at 134.62 153.67 0)
+    (property "Footprint" "Keys:SW_Hybrid_Cherry_MX_Alps_1.50u" (id 2) (at 134.62 153.67 0)
       (effects (font (size 1.27 1.27)) hide)
     )
@@
   (symbol (lib_id "power:GND") (at 247.65 63.5 0) (unit 1)
     (in_bom yes) (on_board yes) (fields_autoplaced)
-    (property "Reference" "#PWR?" (id 0) (at 247.65 69.85 0)
+    (property "Reference" "#PWR0108" (id 0) (at 247.65 69.85 0)
       (effects (font (size 1.27 1.27)) hide)
     )
@@
   (symbol (lib_id "power:+3V3") (at 256.54 55.88 0) (unit 1)
     (in_bom yes) (on_board yes) (fields_autoplaced)
-    (property "Reference" "#PWR?" (id 0) (at 256.54 59.69 0)
+    (property "Reference" "#PWR0109" (id 0) (at 256.54 59.69 0)
       (effects (font (size 1.27 1.27)) hide)
     )
@@
       (effects (font (size 1.27 1.27)) (justify left))
     )
-    (property "Footprint" "Keys:SW_Hybrid_Cherry_MX_Alps_2.00u" (id 2) (at 200.66 140.97 0)
+    (property "Footprint" "Keys:SW_Hybrid_Cherry_MX_Alps_1.50u" (id 2) (at 200.66 140.97 0)
       (effects (font (size 1.27 1.27)) hide)
     )
@@
     )
     (path "/c7440643-8aff-4c0d-9212-6d7e15708ff4"
-      (reference "#PWR?") (unit 1) (value "GND") (footprint "")
+      (reference "#PWR0108") (unit 1) (value "GND") (footprint "")
     )
     (path "/e684eaf6-2a02-4c5b-8ab9-1b8fafe400e0"
-      (reference "#PWR?") (unit 1) (value "+3V3") (footprint "")
+      (reference "#PWR0109") (unit 1) (value "+3V3") (footprint "")
     )
     (path "/c639ccfa-0717-4d61-adf2-d24a823fd40a"
@@
     )
     (path "/9373d9c2-c320-4540-94da-750bd0dff301"
-      (reference "SW4") (unit 1) (value "ShiftL") (footprint "Keys:SW_Hybrid_Cherry_MX_Alps_1.00u")
+      (reference "SW4") (unit 1) (value "ShiftL") (footprint "Keys:SW_Hybrid_Cherry_MX_Alps_1.50u")
     )
     (path "/249113cf-1863-4b8f-a510-599d6a035ab3"
@@
     )
     (path "/7bbbda77-3899-4388-b9dd-2c647177ae2c"
-      (reference "SW25") (unit 1) (value "Space") (footprint "Keys:SW_Hybrid_Cherry_MX_Alps_2.00u")
+      (reference "SW25") (unit 1) (value "Space") (footprint "Keys:SW_Hybrid_Cherry_MX_Alps_1.50u")
     )
     (path "/70e24d71-3182-4333-bd7c-ddee96ee0dfb"
@@
     )
     (path "/3ad64e4b-1f9a-4761-b00b-9fc33ecf740d"
-      (reference "SW30") (unit 1) (value "Space") (footprint "Keys:SW_Hybrid_Cherry_MX_Alps_2.00u")
+      (reference "SW30") (unit 1) (value "Space") (footprint "Keys:SW_Hybrid_Cherry_MX_Alps_6.50u")
     )
     (path "/2a7b7e36-dcf7-484e-904c-bdad9f5071bd"
@@
     )
     (path "/a7658f95-ff45-4aea-be88-ecae8f1b7324"
-      (reference "SW35") (unit 1) (value "Space") (footprint "Keys:SW_Hybrid_Cherry_MX_Alps_2.00u")
+      (reference "SW35") (unit 1) (value "Space") (footprint "Keys:SW_Hybrid_Cherry_MX_Alps_1.50u")
     )
     (path "/557af437-b656-4b19-888b-1d0e32ccd630"
@@
     )
     (path "/ec9b5763-ab78-4b31-bc2d-dd27c7975b6e"
-      (reference "SW51") (unit 1) (value "ShiftR") (footprint "Keys:SW_Hybrid_Cherry_MX_Alps_2.00u")
+      (reference "SW51") (unit 1) (value "ShiftR") (footprint "Keys:SW_Hybrid_Cherry_MX_Alps_1.50u")
     )
     (path "/1f6b193f-62dd-4b0a-af5a-73695a1b0c99"
@@
       (reference "SW62") (unit 1) (value "Special") (footprint "Button_Switch_THT:SW_PUSH-12mm")
     )
+    (path "/6a5ee8a0-bc61-4410-872f-1bdd7f93e634"
+      (reference "Stab1") (unit 1) (value "Stabelizer Enter") (footprint "KeysStable:Stabilizer_Cherry_MX_2.00u")
+    )
+    (path "/1cc8e218-ce15-49a3-b7d7-ba265e0d5f6b"
+      (reference "Stab2") (unit 1) (value "Stabelizer Spacebar") (footprint "KeysStable:Stabilizer_Cherry_MX_6.00u")
+    )
     (path "/7a63fba4-7155-4b02-93ef-c5014077a9f2"
